Commit message: ackermann.gazebo.xacro added the plug in just need to change values.

File: f1tenth_description/gazebo/ackermann.gazebo.xacro (robot description, xacro)
@@ -5,20 +5,21 @@
             filename="gz-sim-ackermann-steering-system"
             name="gz::sim::systems::AckermannSteering">
-        <left_joint>front_left_wheel_joint</left_joint>
-        <left_joint>rear_left_wheel_joint</left_joint>
-        <right_joint>front_right_wheel_joint</right_joint>
-        <right_joint>rear_right_wheel_joint</right_joint>
-        <left_steering_joint>front_left_wheel_steering_joint</left_steering_joint>
-        <right_steering_joint>front_right_wheel_steering_joint</right_steering_joint>
-        <kingpin_width>1.0</kingpin_width>
-        <wheel_base>1.0</wheel_base>
-        <wheel_separation>1.25</wheel_separation>
-        <wheel_radius>0.3</wheel_radius>
-        <steering_limit>0.5</steering_limit>
-        <min_velocity>-1</min_velocity>
-        <max_velocity>1</max_velocity>
-        <min_acceleration>-3</min_acceleration>
-        <max_acceleration>3</max_acceleration>
-      </plugin>
+            <left_joint>front_left_wheel_joint</left_joint>
+            <left_joint>rear_left_wheel_joint</left_joint>
+            <right_joint>front_right_wheel_joint</right_joint>
+            <right_joint>rear_right_wheel_joint</right_joint>
+            <left_steering_joint>front_left_wheel_steering_joint</left_steering_joint>
+            <right_steering_joint>front_right_wheel_steering_joint</right_steering_joint>
+            <!-- TODO: change these numbers so that it is remotely accurate -->
+            <kingpin_width>1.0</kingpin_width>
+            <steering_limit>0.5</steering_limit>
+            <wheel_base>1.0</wheel_base>
+            <wheel_separation>1.25</wheel_separation>
+            <wheel_radius>0.3</wheel_radius>
+            <min_velocity>-1</min_velocity>
+            <max_velocity>1</max_velocity>
+            <min_acceleration>-3</min_acceleration>
+            <max_acceleration>3</max_acceleration>
+        </plugin>
     </gazebo>
 </robot>

File: f1tenth_description/urdf/robot.urdf.xacro (robot description, xacro)
@@ -4,10 +4,8 @@
     <xacro:include filename="$(find f1tenth_description)/urdf/const.xacro" />
     <xacro:include filename="$(find f1tenth_description)/urdf/macro.xacro" />
-<!--    <xacro:property name="sizes_yaml_file" value="$(find f1tenth_description)/config/sizes.xacro" />-->
-<!--    <xacro:property name="sizes" value="${load_yaml(sizes_yaml_file)}" />-->
     <!-- links and joints -->
     <xacro:include filename="$(find f1tenth_description)/urdf/links.xacro" />
     <xacro:include filename="$(find f1tenth_description)/urdf/joints.xacro" />
     <!-- Gazebo stuff -->
-<!--    <xacro:include filename="$(find f1tenth_description)/gazebo/ackermann.gazebo.xacro" />-->
+    <xacro:include filename="$(find f1tenth_description)/gazebo/ackermann.gazebo.xacro" />
 </robot>
