Commit message: Added documentation for macros

File: f1tenth_description/urdf/macro.xacro (robot description, xacro)
@@ -1,4 +1,5 @@
 <?xml version="1.0"?>
 <robot xmlns:xacro="http://www.ros.org/wiki/xacro">
+    <!-- link to full docs: https://github.com/UOA-FSAE/f1tenth/wiki/Description -->
     <xacro:macro name="inertial_sphere" params="mass radius *origin">
         <inertial>
@@ -28,6 +29,28 @@
         </inertial>
     </xacro:macro>
-    <xacro:macro name="wheel" params="name mesh_file radius width mass *origin">
+    <!--
+    https://github.com/UOA-FSAE/f1tenth/wiki/Description#cylinder_link
+    This macro creates a cylinder link
+    params:
+    > name: name of link
+    > mesh_file: link to stl or dae, example `package://f1tenth_description/meshes/chassis_base.stl`
+    > radius: radius of wheel (m)
+    > width: width of wheel (m)
+    > mass: mass of wheel (kg)
+    > *origin: need to include origin tag `<origin xyz="0 0 0" rpy="0 0 0"/>`
+    example: Create a front left wheel with the name of the link being front_left_wheel, mesh located at the
+    f1tenth_description package in the meshes folder called wheel.stl, radius of 0.055m, width of 0.0445m,
+    and mass of 0.09kg with a default origin.
+    ``` XACRO / XML
+    <xacro:cylinder_link name="front_left_wheel" mesh_file="package://f1tenth_description/meshes/wheel.stl"
+                 radius="0.055" width="0.0445" mass="0.09">
+        <origin xyz="0 0 0" rpy="0 0 0"/>
+    <xacro:wheel />
+    ```
+    -->
+    <xacro:macro name="cylinder_link" params="name mesh_file radius width mass *origin">
         <link name="${name}">
+            <!-- Be careful when creating links that you want in gazebo bc you need to have
+             a visual, collision and an inertial component to the link -->
             <visual>
                 <geometry>
@@ -47,5 +70,26 @@
         </link>
     </xacro:macro>
-    <xacro:macro name="chassis_part" params="name mesh_file mass x y z *origin" >
+    <!--
+    https://github.com/UOA-FSAE/f1tenth/wiki/Description#box_link
+    This macro creates a box link
+    params:
+    > name: name of link
+    > mesh_file: link to stl or dae, example `package://f1tenth_description/meshes/chassis_base.stl`
+    > mass: mass of part (kg)
+    > x: length of part (m)
+    > y: height of part (m)
+    > z: width of part (m)
+    > *origin: need to include origin tag `<origin xyz="0 0 0" rpy="0 0 0"/>`
+    example: Create a lower chassis part with the name of the link being lower_chassis, mesh located at the
+    f1tenth_description package in the meshes folder called lower_chassis.stl with a mass of 0.08kg,
+    length of 0.31m, width of 0.183m, and a height of 0.03m with its origin being set to 0 0 0.
+    ``` XACRO / XML
+    <xacro:box_link name="lower_chassis" mesh_file="package://f1tenth_description/meshes/lower_chassis.stl"
+                    x="0.31" y="0.183" z="0.03" mass="0.08">
+        <origin xyz="0 0 0" rpy="0 0 0"/>
+    <xacro:box_link />
+    ```
+    -->
+    <xacro:macro name="box_link" params="name mesh_file mass x y z *origin" >
         <link name="${name}">
             <visual>

Commit message: Created links for the urdf

File: f1tenth_description/urdf/macro.xacro (robot description, xacro)
@@ -48,12 +48,11 @@
     <xacro:wheel />
     ```
+    There is a no mesh option it's called cylinder_link_nomesh that has the same params just with no mesh.
     -->
     <xacro:macro name="cylinder_link" params="name mesh_file radius width mass *origin">
         <link name="${name}">
-            <!-- Be careful when creating links that you want in gazebo bc you need to have
-             a visual, collision and an inertial component to the link -->
             <visual>
                 <geometry>
-                    <mesh filename="mesh_file"/>
+                    <mesh filename="${mesh_file}"/>
                 </geometry>
                 <xacro:insert_block name="origin" />
@@ -61,5 +60,24 @@
             <collision>
                 <geometry>
-                    <mesh filename="mesh_file"/>
+                    <mesh filename="${mesh_file}"/>
+                </geometry>
+                <xacro:insert_block name="origin" />
+            </collision>
+            <xacro:inertial_cylinder mass="${mass}" length="${width}" radius="${radius}">
+                <xacro:insert_block name="origin" />
+            </xacro:inertial_cylinder>
+        </link>
+    </xacro:macro>
+    <xacro:macro name="cylinder_link_nomesh" params="name radius width mass *origin">
+        <link name="${name}">
+            <visual>
+                <geometry>
+                    <cylinder length="${width}" radius="${radius}" />
+                </geometry>
+                <xacro:insert_block name="origin" />
+            </visual>
+            <collision>
+                <geometry>
+                    <cylinder length="${width}" radius="${radius}" />
                 </geometry>
                 <xacro:insert_block name="origin" />
@@ -95,5 +113,5 @@
             <visual>
                 <geometry>
-                    <mesh filename="mesh_file"/>
+                    <mesh filename="${mesh_file}"/>
                 </geometry>
                 <xacro:insert_block name="origin" />
@@ -101,5 +119,5 @@
             <collision>
                 <geometry>
-                    <mesh filename="mesh_file"/>
+                    <mesh filename="${mesh_file}"/>
                 </geometry>
                 <xacro:insert_block name="origin" />

File: f1tenth_description/urdf/robot.urdf.xacro (robot description, xacro)
@@ -4,8 +4,9 @@
     <xacro:include filename="$(find f1tenth_description)/urdf/const.xacro" />
     <xacro:include filename="$(find f1tenth_description)/urdf/macro.xacro" />
-    <xacro:property name="sizes_yaml_file" value="$(find f1tenth_description)/config/sizes.xacro" />
-    <xacro:property name="sizes" value="${load_yaml(sizes_yaml_file)}" />
-    <!-- -->
+<!--    <xacro:property name="sizes_yaml_file" value="$(find f1tenth_description)/config/sizes.xacro" />-->
+<!--    <xacro:property name="sizes" value="${load_yaml(sizes_yaml_file)}" />-->
+    <!-- links and joints -->
+    <xacro:include filename="$(find f1tenth_description)/urdf/links.xacro" />
     <!-- Gazebo stuff -->
-    <xacro:include filename="$(find f1tenth_description)/gazebo/ackermann.gazebo.xacro" />
+<!--    <xacro:include filename="$(find f1tenth_description)/gazebo/ackermann.gazebo.xacro" />-->
 </robot>

Commit message: refactor: simplify collision geometry of the robot wheels

File: f1tenth_description/urdf/macro.xacro (robot description, xacro)
@@ -61,6 +61,5 @@
             <collision>
                 <geometry>
-                    <mesh filename="${mesh_file}"
-                        scale="0.001 0.001 0.001"/>
+                    <cylinder length="${width}" radius="${radius}" />
                 </geometry>
                 <xacro:insert_block name="origin" />
