Commit message: rsp stuff

File: f1tenth_description/urdf/joints.xacro (robot description, xacro)
@@ -3,6 +3,6 @@
     <!-- Steering joints -->
     <joint name="front_left_wheel_steering_joint" type="revolute">
-        <child>front_left_wheel_steering_link</child>
-        <parent>base_link</parent>
+        <child link="front_left_wheel_steering_link" />
+        <parent link="base_link" />
         <axis xyz="0 0 1" />
         <limit lower="-0.6" upper="+0.6"
@@ -10,6 +10,6 @@
     </joint>
     <joint name="front_right_wheel_steering_joint" type="revolute">
-        <child>front_right_wheel_steering_link</child>
-        <parent>base_link</parent>
+        <child link="front_right_wheel_steering_link" />
+        <parent link="base_link" />
         <axis xyz="0 0 1" />
         <limit lower="-0.6" upper="+0.6"
@@ -18,21 +18,21 @@
     <!-- Drive joints -->
     <joint name="front_left_wheel_joint" type="continuous">
-        <child>front_left_wheel</child>
-        <parent>front_left_wheel_steering_link</parent>
+        <child link="front_left_wheel" />
+        <parent link="front_left_wheel_steering_link" />
         <axis xyz="0 0 1" />
     </joint>
     <joint name="front_right_wheel_joint" type="continuous">
-        <child>front_right_wheel</child>
-        <parent>front_right_wheel_steering_link</parent>
+        <child link="front_right_wheel" />
+        <parent link="front_right_wheel_steering_link" />
         <axis xyz="0 0 1" />
     </joint>
     <joint name="rear_left_wheel_joint" type="continuous">
-        <child>rear_left_wheel</child>
-        <parent>base_link</parent>
+        <child link="rear_left_wheel" />
+        <parent link="base_link" />
         <axis xyz="0 0 1" />
     </joint>
     <joint name="rear_right_wheel_joint" type="continuous">
-        <child>rear_right_wheel</child>
-        <parent>base_link</parent>
+        <child link="rear_right_wheel" />
+        <parent link="base_link" />
         <axis xyz="0 0 1" />
     </joint>

File: f1tenth_description/urdf/links.xacro (robot description, xacro)
@@ -15,5 +15,5 @@
         <origin xyz="0 0 0" rpy="0 0 0"/>
     </xacro:cylinder_link>
-    <xacro:cylinder_link name="rear_left_wheel" mesh_file="package://f1tenth_description/meshes/wheel.stl"
+    <xacro:cylinder_link name="rear_right_wheel" mesh_file="package://f1tenth_description/meshes/wheel.stl"
                  radius="0.055" width="0.0445" mass="0.09">
         <origin xyz="0 0 0" rpy="0 0 0"/>
@@ -29,7 +29,7 @@
     </xacro:cylinder_link_nomesh>
     <!-- Chassis -->
-    <xacro:box_link name="lower_chassis" mesh_file="package://f1tenth_description/meshes/lower_chassis.stl"
-                    x="0.31" y="0.183" z="0.03" mass="0.08">
-        <origin xyz="0 0 0" rpy="0 0 0"/>
-    </xacro:box_link>
+<!--    <xacro:box_link name="lower_chassis" mesh_file="package://f1tenth_description/meshes/lower_chassis.stl"-->
+<!--                    x="0.31" y="0.183" z="0.03" mass="0.08">-->
+<!--        <origin xyz="0 0 0" rpy="0 0 0"/>-->
+<!--    </xacro:box_link>-->
 </robot>

Commit message: I HATE FLAGS WITH A PASSION!

File: f1tenth_description/urdf/joints.xacro (robot description, xacro)
@@ -8,4 +8,5 @@
         <limit lower="-0.6" upper="+0.6"
                velocity="1.0" effort="25" />
+        <origin xyz="0.1575 0.1025 0.055" rpy="0 0 0"/>
     </joint>
     <joint name="front_right_wheel_steering_joint" type="revolute">
@@ -15,4 +16,5 @@
         <limit lower="-0.6" upper="+0.6"
                velocity="1.0" effort="25" />
+        <origin xyz="0.1575 -0.1025 0.055" rpy="0 0 0"/>
     </joint>
     <!-- Drive joints -->
@@ -20,20 +22,28 @@
         <child link="front_left_wheel" />
         <parent link="front_left_wheel_steering_link" />
-        <axis xyz="0 0 1" />
+        <axis xyz="0 1 0" />
     </joint>
     <joint name="front_right_wheel_joint" type="continuous">
         <child link="front_right_wheel" />
         <parent link="front_right_wheel_steering_link" />
-        <axis xyz="0 0 1" />
+        <axis xyz="0 1 0" />
     </joint>
     <joint name="rear_left_wheel_joint" type="continuous">
         <child link="rear_left_wheel" />
         <parent link="base_link" />
-        <axis xyz="0 0 1" />
+        <axis xyz="0 1 0" />
+        <origin xyz="-0.1575 0.1025 0.055" rpy="0 0 0"/>
     </joint>
     <joint name="rear_right_wheel_joint" type="continuous">
         <child link="rear_right_wheel" />
         <parent link="base_link" />
-        <axis xyz="0 0 1" />
+        <axis xyz="0 1 0" />
+        <origin xyz="-0.1575 -0.1025 0.055" rpy="0 0 0"/>
+    </joint>
+    <!-- Chassis Joints-->
+    <joint name="base_link_to_lower_chassis" type="fixed">
+        <child link="lower_chassis" />
+        <parent link="base_link" />
+        <origin xyz="-0.155 0.09 0.055" rpy="0 0 0"/>
     </joint>
 </robot>

File: f1tenth_description/urdf/links.xacro (robot description, xacro)
@@ -5,17 +5,17 @@
     <xacro:cylinder_link name="front_left_wheel" mesh_file="package://f1tenth_description/meshes/wheel.stl"
                  radius="0.055" width="0.0445" mass="0.09">
-        <origin xyz="0 0 0" rpy="0 0 0"/>
+        <origin xyz="0 0 0" rpy="${-pi/2} 0 0"/>
     </xacro:cylinder_link>
     <xacro:cylinder_link name="front_right_wheel" mesh_file="package://f1tenth_description/meshes/wheel.stl"
                  radius="0.055" width="0.0445" mass="0.09">
-        <origin xyz="0 0 0" rpy="0 0 0"/>
+        <origin xyz="0 0 0" rpy="${pi/2} 0 0"/>
     </xacro:cylinder_link>
     <xacro:cylinder_link name="rear_left_wheel" mesh_file="package://f1tenth_description/meshes/wheel.stl"
                  radius="0.055" width="0.0445" mass="0.09">
-        <origin xyz="0 0 0" rpy="0 0 0"/>
+        <origin xyz="0 0 0" rpy="${-pi/2} 0 0"/>
     </xacro:cylinder_link>
     <xacro:cylinder_link name="rear_right_wheel" mesh_file="package://f1tenth_description/meshes/wheel.stl"
                  radius="0.055" width="0.0445" mass="0.09">
-        <origin xyz="0 0 0" rpy="0 0 0"/>
+        <origin xyz="0 0 0" rpy="${pi/2} 0 0"/>
     </xacro:cylinder_link>
     <!-- Drive train -->
@@ -29,7 +29,7 @@
     </xacro:cylinder_link_nomesh>
     <!-- Chassis -->
-<!--    <xacro:box_link name="lower_chassis" mesh_file="package://f1tenth_description/meshes/lower_chassis.stl"-->
-<!--                    x="0.31" y="0.183" z="0.03" mass="0.08">-->
-<!--        <origin xyz="0 0 0" rpy="0 0 0"/>-->
-<!--    </xacro:box_link>-->
+    <xacro:box_link name="lower_chassis" mesh_file="package://f1tenth_description/meshes/chassis_base.stl"
+                    x="0.31" y="0.183" z="0.03" mass="0.08">
+        <origin xyz="0 0 0" rpy="0 0 ${-pi/2}"/>
+    </xacro:box_link>
 </robot>

File: f1tenth_description/urdf/macro.xacro (robot description, xacro)
@@ -54,5 +54,6 @@
             <visual>
                 <geometry>
-                    <mesh filename="${mesh_file}"/>
+                    <mesh filename="${mesh_file}"
+                        scale="0.001 0.001 0.001"/>
                 </geometry>
                 <xacro:insert_block name="origin" />
@@ -60,5 +61,6 @@
             <collision>
                 <geometry>
-                    <mesh filename="${mesh_file}"/>
+                    <mesh filename="${mesh_file}"
+                        scale="0.001 0.001 0.001"/>
                 </geometry>
                 <xacro:insert_block name="origin" />
@@ -113,5 +115,6 @@
             <visual>
                 <geometry>
-                    <mesh filename="${mesh_file}"/>
+                    <mesh filename="${mesh_file}"
+                        scale="0.001 0.001 0.001"/>
                 </geometry>
                 <xacro:insert_block name="origin" />
@@ -119,5 +122,6 @@
             <collision>
                 <geometry>
-                    <mesh filename="${mesh_file}"/>
+                    <mesh filename="${mesh_file}"
+                        scale="0.001 0.001 0.001"/>
                 </geometry>
                 <xacro:insert_block name="origin" />

Commit message: Added Lidar to thingy

File: f1tenth_description/urdf/joints.xacro (robot description, xacro)
@@ -47,3 +47,9 @@
         <origin xyz="-0.155 0.09 0.055" rpy="0 0 0"/>
     </joint>
+    <!-- Sensor Joints -->
+    <joint name="hokuyo_10lx_lidar_joint" type="fixed">
+        <child link="hokuyo_10lx_lidar_link" />
+        <parent link="base_link" />
+        <origin xyz="0.1 0 0.15" rpy="0 0 0"/>
+    </joint>
 </robot>

File: f1tenth_description/urdf/links.xacro (robot description, xacro)
@@ -33,3 +33,8 @@
         <origin xyz="0 0 0" rpy="0 0 ${-pi/2}"/>
     </xacro:box_link>
+    <!-- Sensor links -->
+    <xacro:cylinder_link_nomesh name="hokuyo_10lx_lidar_link"
+                    radius="0.05" width="0.08" mass="0.05">
+      <origin xyz="0 0 0" rpy="0 0 0"/>
+    </xacro:cylinder_link_nomesh>
 </robot>

File: f1tenth_description/urdf/robot.urdf.xacro (robot description, xacro)
@@ -4,8 +4,10 @@
     <xacro:include filename="$(find f1tenth_description)/urdf/const.xacro" />
     <xacro:include filename="$(find f1tenth_description)/urdf/macro.xacro" />
+    <xacro:include filename="$(find f1tenth_description)/gazebo/lidar.gazebo.xacro" />
     <!-- links and joints -->
     <xacro:include filename="$(find f1tenth_description)/urdf/links.xacro" />
     <xacro:include filename="$(find f1tenth_description)/urdf/joints.xacro" />
-    <!-- Gazebo stuff -->
+<!--    &lt;!&ndash; Gazebo stuff &ndash;&gt;-->
+<!--    <xacro:include filename="$(find f1tenth_description)/gazebo/lidar.gazebo.xacro" />-->
     <xacro:include filename="$(find f1tenth_description)/gazebo/ackermann.gazebo.xacro" />
     <xacro:include filename="$(find f1tenth_description)/gazebo/odometry.gazebo.xacro" />

Commit message: Add cardboard

File: f1tenth_description/urdf/joints.xacro (robot description, xacro)
@@ -42,4 +42,9 @@
     </joint>
     <!-- Chassis Joints-->
+    <joint name="base_link_to_box" type="fixed">
+        <child link="box_visual" />
+        <parent link="base_link" />
+        <origin xyz="-0.1554 0.09 0.2" rpy="0 0 0"/>
+    </joint>
     <joint name="base_link_to_lower_chassis" type="fixed">
         <child link="lower_chassis" />

File: f1tenth_description/urdf/links.xacro (robot description, xacro)
@@ -30,7 +30,10 @@
     <!-- Chassis -->
     <xacro:box_link name="lower_chassis" mesh_file="package://f1tenth_description/meshes/chassis_base.stl"
-                    x="0.31" y="0.183" z="0.03" mass="0.08">
+                    x="0.03" y="0.183" z="0.31 " mass="0.08">
         <origin xyz="0 0 0" rpy="0 0 ${-pi/2}"/>
     </xacro:box_link>
+    <xacro:box_link_nomesh name='box_visual' x="0.03 " y="0.183" z="0.31" mass="0.001">
+        <origin xyz="0 -0.0915 0" rpy="0 0 0"/>
+    </xacro:box_link_nomesh >
     <!-- Sensor links -->
     <xacro:cylinder_link_nomesh name="hokuyo_10lx_lidar_link"

File: f1tenth_description/urdf/macro.xacro (robot description, xacro)
@@ -131,3 +131,22 @@
         </link>
     </xacro:macro>
+  <xacro:macro name="box_link_nomesh" params="name x y z mass *origin">
+        <link name="${name}">
+            <visual>
+                <geometry>
+                    <box size='${x} ${y} ${z}' />
+                </geometry>
+                <xacro:insert_block name="origin" />
+            </visual>
+            <collision>
+                <geometry>
+                    <box size='${x} ${y} ${z}' />
+                </geometry>
+                <xacro:insert_block name="origin" />
+            </collision>
+            <xacro:inertial_box mass="${mass}" x="${x}" y="${y}" z="${z}">
+                <xacro:insert_block name="origin" />
+            </xacro:inertial_box>
+        </link>
+    </xacro:macro>
 </robot>

Commit message: make cardboard white and remove aruco image padding

File: f1tenth_description/urdf/joints.xacro (robot description, xacro)
@@ -67,5 +67,5 @@
         <gazebo>
             <joint name="aruco_marker_joint" type="fixed">
-                <pose relative_to="box_visual">0 0 0 0 0 0</pose>
+                <pose relative_to="box_visual">0 0 0 0 0 0</pose> <!-- This doesn't do anything -->
                 <child>aruco_link</child>
                 <parent>box_visual</parent>

File: f1tenth_description/urdf/links.xacro (robot description, xacro)
@@ -37,4 +37,15 @@
         <origin xyz="0 -0.0915 0" rpy="0 0 0"/>
     </xacro:box_link_nomesh >
+    <!-- Give box visual white color -->
+    <gazebo reference="box_visual">
+        <visual>
+            <material>
+                <emissive>1 1 1 1</emissive>
+                <diffuse>1 1 1 1</diffuse>
+                <specular>1 1 1 1</specular>
+                <ambient>1 1 1 1</ambient>
+            </material>
+        </visual>
+    </gazebo>
     <!-- Sensor links -->
     <xacro:cylinder_link_nomesh name="hokuyo_10lx_lidar_link"
@@ -49,5 +60,5 @@
     <xacro:if value="${add_aruco}">
         <xacro:include filename="$(find f1tenth_description)/sdf/aruco_marker/model.urdf.xacro" />
-        <xacro:aruco_marker xyz="-0.20 0 0.183" rpy="0 0 0"/>
+        <xacro:aruco_marker xyz="-0.1705 0 0.183" rpy="0 0 0"/>
     </xacro:if>
 </robot>
