Commit message: removed need for colour tag now that mesh is implimented in wheel macro

File: f1tenth_description/urdf/const.xacro (robot description, xacro)
@@ -1,3 +1,16 @@
 <?xml version="1.0"?>
 <robot xmlns:xacro="http://www.ros.org/wiki/xacro">
+    <!-- Global -->
+    <xacro:property name="robot_name" value="f1tenth" />
+    <!-- Wheels -->
+    <xacro:property name="wheel_diameter" value="0.11" />
+    <xacro:property name="wheel_width" value="0.0445" />
+    <!-- Chassis -->
+    <xacro:property name="chassis_width" value="0.18" />
+    <xacro:property name="chassis_length" value="0.1" />
+    <xacro:property name="chassis_height" value="0.09" />
+    <!-- Joint placement -->
+    <xacro:property name="chassis_to_wheel_x" value="${0.31 /2}" />
+    <xacro:property name="chassis_to_wheel_y" value="${0.005+ (wheel_width /2) + (chassis_width /2)}" />
+    <xacro:property name="chassis_to_wheel_z" value="${wheel_diameter /2}" />
 </robot>

File: f1tenth_description/urdf/macro.xacro (robot description, xacro)
@@ -28,5 +28,5 @@
         </inertial>
     </xacro:macro>
-    <xacro:macro name="wheel" params="name mesh_file radius width mass colour *origin">
+    <xacro:macro name="wheel" params="name mesh_file radius width mass *origin">
         <link name="${name}">
             <visual>

Commit message: feat: namespace lidar dynamically

File: f1tenth_description/urdf/const.xacro (robot description, xacro)
@@ -2,5 +2,7 @@
 <robot xmlns:xacro="http://www.ros.org/wiki/xacro">
     <!-- Global -->
-    <xacro:property name="robot_name" value="f1tenth" />
+    <xacro:arg name="robot_name" default="f1tenth"/>
+    <xacro:property name="robot_name" value="$(arg robot_name)" />
+    <!-- <xacro:property name="params_path" value="$(arg params_path)"/> -->
     <!-- Wheels -->
     <xacro:property name="wheel_diameter" value="0.11" />

File: f1tenth_description/urdf/macro.xacro (robot description, xacro)
@@ -120,5 +120,5 @@
                 <xacro:insert_block name="origin" />
             </visual>
-            <collision>
+            <!-- <collision>
                 <geometry>
                     <mesh filename="${mesh_file}"
@@ -126,5 +126,5 @@
                 </geometry>
                 <xacro:insert_block name="origin" />
-            </collision>
+            </collision> -->
             <xacro:inertial_box mass="${mass}" x="${x}" y="${y}" z="${z}">
                 <xacro:insert_block name="origin" />

Commit message: add camera and marker to robot description

File: f1tenth_description/urdf/const.xacro (robot description, xacro)
@@ -4,4 +4,8 @@
     <xacro:arg name="robot_name" default="f1tenth"/>
     <xacro:property name="robot_name" value="$(arg robot_name)" />
+    <xacro:arg name="add_camera" default="false"/>
+    <xacro:property name="add_camera" value="$(arg add_camera)" />
+    <xacro:arg name="add_aruco" default="false"/>
+    <xacro:property name="add_aruco" value="$(arg add_aruco)" />
     <!-- <xacro:property name="params_path" value="$(arg params_path)"/> -->
     <!-- Wheels -->

File: f1tenth_description/urdf/joints.xacro (robot description, xacro)
@@ -33,5 +33,5 @@
         <parent link="base_link" />
         <axis xyz="0 1 0" />
-        <origin xyz="-0.1575 0.1025 0.055" rpy="0 0 0"/>
+        <origin xyz="-0.1575 0.1025 0.055" rpy="0 0 0" />
     </joint>
     <joint name="rear_right_wheel_joint" type="continuous">
@@ -39,5 +39,5 @@
         <parent link="base_link" />
         <axis xyz="0 1 0" />
-        <origin xyz="-0.1575 -0.1025 0.055" rpy="0 0 0"/>
+        <origin xyz="-0.1575 -0.1025 0.055" rpy="0 0 0" />
     </joint>
     <!-- Chassis Joints-->
@@ -45,10 +45,10 @@
         <child link="box_visual" />
         <parent link="base_link" />
-        <origin xyz="-0.1554 0.09 0.2" rpy="0 0 0"/>
+        <origin xyz="-0.1554 0.09 0.2" rpy="0 0 0" />
     </joint>
     <joint name="base_link_to_lower_chassis" type="fixed">
         <child link="lower_chassis" />
         <parent link="base_link" />
-        <origin xyz="-0.155 0.09 0.055" rpy="0 0 0"/>
+        <origin xyz="-0.155 0.09 0.055" rpy="0 0 0" />
     </joint>
     <!-- Sensor Joints -->
@@ -56,5 +56,5 @@
         <child link="hokuyo_10lx_lidar_link" />
         <parent link="base_link" />
-        <origin xyz="0.1 0 0.15" rpy="0 0 0"/>
+        <origin xyz="0.1 0 0.15" rpy="0 0 0" />
     </joint>
     <joint name="imu_sensor_joint" type="fixed">
@@ -63,3 +63,12 @@
         <origin xyz="0 0 0" rpy="0 0 0"/>
     </joint>
+    <xacro:if value="${add_aruco}">
+        <gazebo>
+            <joint name="aruco_marker_joint" type="fixed">
+                <pose relative_to="box_visual">0 0 0 0 0 0</pose>
+                <child>aruco_link</child>
+                <parent>box_visual</parent>
+            </joint>
+        </gazebo>
+    </xacro:if>
 </robot>

File: f1tenth_description/urdf/links.xacro (robot description, xacro)
@@ -46,3 +46,8 @@
         <origin xyz="0 0 0" rpy="0 0 0"/>
     </link>
+    <!-- AruCo marker -->
+    <xacro:if value="${add_aruco}">
+        <xacro:include filename="$(find f1tenth_description)/sdf/aruco_marker/model.urdf.xacro" />
+        <xacro:aruco_marker xyz="-0.20 0 0.183" rpy="0 0 0"/>
+    </xacro:if>
 </robot>

File: f1tenth_description/urdf/robot.urdf.xacro (robot description, xacro)
@@ -9,4 +9,5 @@
     <xacro:include filename="$(find f1tenth_description)/urdf/links.xacro" />
     <xacro:include filename="$(find f1tenth_description)/urdf/joints.xacro" />
+    <xacro:include filename="$(find f1tenth_description)/urdf/d435.xacro" />
     <!-- Gazebo stuff -->
     <xacro:include filename="$(find f1tenth_description)/gazebo/ackermann.gazebo.xacro" />

Commit message: take camera name in macro

File: f1tenth_description/urdf/const.xacro (robot description, xacro)
@@ -4,4 +4,6 @@
     <xacro:arg name="robot_name" default="f1tenth"/>
     <xacro:property name="robot_name" value="$(arg robot_name)" />
+    <xacro:arg name="camera_name" default="d435"/>
+    <xacro:property name="camera_name" value="$(arg camera_name)" />
     <xacro:arg name="add_camera" default="false"/>
     <xacro:property name="add_camera" value="$(arg add_camera)" />

File: f1tenth_description/urdf/joints.xacro (robot description, xacro)
@@ -63,4 +63,5 @@
         <origin xyz="0 0 0" rpy="0 0 0"/>
     </joint>
+    <!-- Add AruCo marker  -->
     <xacro:if value="${add_aruco}">
         <gazebo>

Commit message: add stereo camera macro

File: f1tenth_description/urdf/const.xacro (robot description, xacro)
@@ -6,4 +6,6 @@
     <xacro:arg name="camera_name" default="d435"/>
     <xacro:property name="camera_name" value="$(arg camera_name)" />
+    <xacro:arg name="stereo_camera_name" default="zed2"/>
+    <xacro:property name="stereo_camera_name" value="$(arg stereo_camera_name)" />
     <xacro:arg name="add_camera" default="false"/>
     <xacro:property name="add_camera" value="$(arg add_camera)" />

File: f1tenth_description/urdf/d435.xacro (robot description, xacro)
@@ -4,8 +4,8 @@
   <xacro:include filename="$(find realsense2_description)/urdf/_d435.urdf.xacro" />
   <xacro:if value="${add_camera}">
-    <xacro:sensor_d435 gazebo="true" name="${camera_name}" parent="base_link"
-      use_nominal_extrinsics="true"
+    <xacro:sensor_d435 gazebo="true" robot_name="${robot_name}"
+      name="${camera_name}" parent="base_link" use_nominal_extrinsics="false"
       enable_infra1="false" enable_infra2="false" enable_color="true" enable_depth="true"
-      color_width="1920" color_height="1080" color_fps="30"
+      color_width="1280" color_height="720" color_fps="30"
       depth_width="1280" depth_height="720" depth_fps="30">
       <origin xyz="0 0 0.3" rpy="0 0 0" />

File: f1tenth_description/urdf/robot.urdf.xacro (robot description, xacro)
@@ -9,4 +9,5 @@
     <xacro:include filename="$(find f1tenth_description)/urdf/joints.xacro" />
     <xacro:include filename="$(find f1tenth_description)/urdf/d435.xacro" />
+    <!-- <xacro:include filename="$(find f1tenth_description)/urdf/zed2.xacro" /> -->
     <!-- Gazebo stuff -->
     <xacro:include filename="$(find f1tenth_description)/gazebo/ackermann.gazebo.xacro" />

Commit message: add stereo camera macro

File: f1tenth_description/urdf/const.xacro (robot description, xacro)
@@ -6,4 +6,6 @@
     <xacro:arg name="camera_name" default="d435"/>
     <xacro:property name="camera_name" value="$(arg camera_name)" />
+    <xacro:arg name="stereo_camera_name" default="zed2"/>
+    <xacro:property name="stereo_camera_name" value="$(arg stereo_camera_name)" />
     <xacro:arg name="add_camera" default="false"/>
     <xacro:property name="add_camera" value="$(arg add_camera)" />

File: f1tenth_description/urdf/robot.urdf.xacro (robot description, xacro)
@@ -10,4 +10,5 @@
     <xacro:include filename="$(find f1tenth_description)/urdf/joints.xacro" />
     <xacro:include filename="$(find f1tenth_description)/urdf/d435.xacro" />
+    <!-- <xacro:include filename="$(find f1tenth_description)/urdf/zed2.xacro" /> -->
     <!-- Gazebo stuff -->
     <xacro:include filename="$(find f1tenth_description)/gazebo/ackermann.gazebo.xacro" />

Commit message: add switch for stereo and monocular

File: f1tenth_description/urdf/const.xacro (robot description, xacro)
@@ -12,5 +12,6 @@
     <xacro:arg name="add_aruco" default="false"/>
     <xacro:property name="add_aruco" value="$(arg add_aruco)" />
-    <!-- <xacro:property name="params_path" value="$(arg params_path)"/> -->
+    <xacro:arg name="use_stereo" default="false"/>
+    <xacro:property name="use_stereo" value="$(arg use_stereo)" />
     <!-- Wheels -->
     <xacro:property name="wheel_diameter" value="0.11" />

File: f1tenth_description/urdf/robot.urdf.xacro (robot description, xacro)
@@ -9,6 +9,10 @@
     <xacro:include filename="$(find f1tenth_description)/urdf/links.xacro" />
     <xacro:include filename="$(find f1tenth_description)/urdf/joints.xacro" />
-    <xacro:include filename="$(find f1tenth_description)/urdf/d435.xacro" />
-    <!-- <xacro:include filename="$(find f1tenth_description)/urdf/zed2.xacro" /> -->
+    <xacro:if value="$(arg use_stereo)">
+        <xacro:include filename="$(find f1tenth_description)/urdf/zed2.xacro" />
+    </xacro:if>
+    <xacro:unless value="$(arg use_stereo)">
+        <xacro:include filename="$(find f1tenth_description)/urdf/d435.xacro" />
+    </xacro:unless>
     <!-- Gazebo stuff -->
     <xacro:include filename="$(find f1tenth_description)/gazebo/ackermann.gazebo.xacro" />

Commit message: add switch for stereo and monocular

File: f1tenth_description/urdf/const.xacro (robot description, xacro)
@@ -12,5 +12,6 @@
     <xacro:arg name="add_aruco" default="false"/>
     <xacro:property name="add_aruco" value="$(arg add_aruco)" />
-    <!-- <xacro:property name="params_path" value="$(arg params_path)"/> -->
+    <xacro:arg name="use_stereo" default="false"/>
+    <xacro:property name="use_stereo" value="$(arg use_stereo)" />
     <!-- Wheels -->
     <xacro:property name="wheel_diameter" value="0.11" />

File: f1tenth_description/urdf/robot.urdf.xacro (robot description, xacro)
@@ -8,6 +8,10 @@
     <xacro:include filename="$(find f1tenth_description)/urdf/links.xacro" />
     <xacro:include filename="$(find f1tenth_description)/urdf/joints.xacro" />
-    <xacro:include filename="$(find f1tenth_description)/urdf/d435.xacro" />
-    <!-- <xacro:include filename="$(find f1tenth_description)/urdf/zed2.xacro" /> -->
+    <xacro:if value="$(arg use_stereo)">
+        <xacro:include filename="$(find f1tenth_description)/urdf/zed2.xacro" />
+    </xacro:if>
+    <xacro:unless value="$(arg use_stereo)">
+        <xacro:include filename="$(find f1tenth_description)/urdf/d435.xacro" />
+    </xacro:unless>
     <!-- Gazebo stuff -->
     <xacro:include filename="$(find f1tenth_description)/gazebo/ackermann.gazebo.xacro" />

File: f1tenth_description/urdf/zed2.xacro (robot description, xacro)
@@ -6,7 +6,8 @@
     <xacro:zed_camera parent="base_link"
       gazebo="true" robot_name="$(arg robot_name)"
+      image_width="1280" image_height="720" fps="30"
       name="$(arg stereo_camera_name)" model="zed2"
       custom_baseline="false" enable_gnss="false">
-      <origin xyz="0 0 0.3" rpy="0 0 0" />
+      <origin xyz="0 0 0.4" rpy="0 0 0" />
     </xacro:zed_camera>
   </xacro:if>
