Commit message: make cardboard white and remove aruco image padding

File: f1tenth_description/sdf/aruco_marker/model.urdf.xacro (robot description, xacro)
@@ -28,7 +28,15 @@
             <specular>0.4 0.4 0.4 1</specular>
             <ambient>1 1 1 1</ambient>
+            <!-- <emissive>0.1 0.1 0.1 1</emissive> -->
             <pbr>
               <metal>
-                <albedo_map>$(find f1tenth_description)/sdf/aruco_marker/materials/textures/marker_padded.png</albedo_map>
+                <albedo_map>$(find f1tenth_description)/sdf/aruco_marker/materials/textures/marker.png</albedo_map>
+                <!-- <roughness_map>$(find f1tenth_description)/sdf/aruco_marker/materials/textures/marker_padded.png</roughness_map> -->
+                <!-- <metalness_map>$(find f1tenth_description)/sdf/aruco_marker/materials/textures/marker_padded.png</metalness_map> -->
+                <!-- <environment_map>$(find f1tenth_description)/sdf/aruco_marker/materials/textures/marker_padded.png</environment_map> -->
+                <!-- <normal_map>$(find f1tenth_description)/sdf/aruco_marker/materials/textures/marker_padded.png</normal_map> -->
+                <!-- <ambient_occlusion_map>$(find f1tenth_description)/sdf/aruco_marker/materials/textures/marker_padded.png</ambient_occlusion_map> -->
+                <!-- <light_map>$(find f1tenth_description)/sdf/aruco_marker/materials/textures/marker_padded.png</light_map> -->
+                <!-- <emissive_map>$(find f1tenth_description)/sdf/aruco_marker/materials/textures/marker_padded.png</emissive_map> -->
                 <metalness>0</metalness>
               </metal>

File: f1tenth_description/urdf/d435.xacro (robot description, xacro)
@@ -5,7 +5,7 @@
   <xacro:if value="${add_camera}">
     <xacro:sensor_d435 gazebo="true" robot_name="${robot_name}"
-      name="${camera_name}" parent="base_link" use_nominal_extrinsics="false"
+      name="${camera_name}" parent="base_link" use_nominal_extrinsics="true"
       enable_infra1="false" enable_infra2="false" enable_color="true" enable_depth="true"
-      color_width="1280" color_height="720" color_fps="30"
+      color_width="1920" color_height="1080" color_fps="30"
       depth_width="1280" depth_height="720" depth_fps="30">
       <origin xyz="0 0 0.3" rpy="0 0 0" />

File: f1tenth_description/urdf/joints.xacro (robot description, xacro)
@@ -62,5 +62,5 @@
         <gazebo>
             <joint name="aruco_marker_joint" type="fixed">
-                <pose relative_to="box_visual">0 0 0 0 0 0</pose>
+                <pose relative_to="box_visual">0 0 0 0 0 0</pose> <!-- This doesn't do anything -->
                 <child>aruco_link</child>
                 <parent>box_visual</parent>

File: f1tenth_description/urdf/links.xacro (robot description, xacro)
@@ -36,4 +36,15 @@
         <origin xyz="0 -0.0915 0" rpy="0 0 0"/>
     </xacro:box_link_nomesh >
+    <!-- Give box visual white color -->
+    <gazebo reference="box_visual">
+        <visual>
+            <material>
+                <emissive>1 1 1 1</emissive>
+                <diffuse>1 1 1 1</diffuse>
+                <specular>1 1 1 1</specular>
+                <ambient>1 1 1 1</ambient>
+            </material>
+        </visual>
+    </gazebo>
     <!-- Sensor links -->
     <xacro:cylinder_link_nomesh name="hokuyo_10lx_lidar_link"
@@ -44,5 +55,5 @@
     <xacro:if value="${add_aruco}">
         <xacro:include filename="$(find f1tenth_description)/sdf/aruco_marker/model.urdf.xacro" />
-        <xacro:aruco_marker xyz="-0.20 0 0.183" rpy="0 0 0"/>
+        <xacro:aruco_marker xyz="-0.1705 0 0.183" rpy="0 0 0"/>
     </xacro:if>
 </robot>
